File: FunKey.kicad_pcb (KiCad board)
At the start: 4 copper layers, 42 x 32 mm, 218 parts, among them J1 MH3-1-0.05, J2 U02-BFD3111B0-009, J3 DF37NB-24DS-0.4V(51), J4 TF-110, J5 SM02B-SRSS-TB, Q1 IRLML2244TRPBF, U1 PCAL6416AHF,128, U2 PAM8301AAF, U3 V3S, U4 SY8088AAC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

Commit message: Revision F with 0.3mm increased length speaker tabs and added drills in the side button corners to make cutout square
Signed-off-by: Michel-FK <michel.stempin@funkey-project.com>
Routing:
- net GND: track 20.9 -> 57.4 mm
Other:
- outline, holes or cut-outs redrawn
- board text added: "20210322"
- board text added: "F"
- board text added: "c 2017-2021, Michel Stempin All rights reserved."
- board text removed: "20200614"
- board text removed: "E"
- board text removed: "c 2017-2020, Michel Stempin All rights reserved."
